Commit message: fixed bug

File: legged_gym/resources/robots/Lite3/urdf/Lite3.urdf (robot description, URDF)
Before this commit: robot Xiaoli, 17 links, 16 joints
Links:
- link FL_HIP: geometry collision mesh filename=../meshes/fl_hip.STL; visual mesh filename=../meshes/fl_hip_hull.STL
- link FL_THIGH: geometry collision mesh filename=../meshes/fl_thigh.STL; visual mesh filename=../meshes/fl_thigh_hull.STL
- link FR_HIP: geometry collision mesh filename=../meshes/fr_hip.STL; visual mesh filename=../meshes/fr_hip_hull.STL
- link FR_THIGH: geometry collision mesh filename=../meshes/fr_thigh.STL; visual mesh filename=../meshes/fr_thigh_hull.STL
- link HL_HIP: geometry collision mesh filename=../meshes/hl_hip.STL; visual mesh filename=../meshes/hl_hip_hull.STL
- link HL_THIGH: geometry collision mesh filename=../meshes/hl_thigh.STL; visual mesh filename=../meshes/hl_thigh_hull.STL
- link HR_HIP: geometry collision mesh filename=../meshes/hr_hip.STL; visual mesh filename=../meshes/hr_hip_hull.STL
- link HR_THIGH: geometry collision mesh filename=../meshes/hr_thigh.STL; visual mesh filename=../meshes/hr_thigh_hull.STL
- link TORSO: geometry collision mesh filename=../meshes/torso.STL; visual mesh filename=../meshes/torso_hull.STL
